Commit message: Add files via upload

File: Pydrake Model/models/FPVDrone.urdf.xacro (robot description, xacro)
@@ -1,4 +1,4 @@
 <?xml version="1.0"?>
-<robot name="copter" xmlns:xacro="http://ros.org/wiki/xacro" xmlns:drake="http://mit.edu">
+<robot name="drone" xmlns:xacro="http://ros.org/wiki/xacro" xmlns:drake="http://mit.edu">
   <!-- File Conventions
     - mass (kg)
@@ -76,6 +76,6 @@
   </material>
   <!-- #endregion -->
-  <!-- #region Copter Base -->
-  <link name="copter_base">
+  <!-- #region Drone Base -->
+  <link name="drone_base">
     <inertial>
       <origin xyz="${zero_origin}" rpy="${zero_rpy}"/>
@@ -98,6 +98,6 @@
   </link>
   <!-- #endregion -->
-  <!-- #region Copter Arms -->
-  <link name="copter_arm_1">
+  <!-- #region Drone Arms -->
+  <link name="drone_arm_1">
     <inertial>
       <origin xyz="${arm_origin}" rpy="${zero_rpy}"/>
@@ -119,5 +119,5 @@
     </collision>
   </link>
-  <link name="copter_arm_2">
+  <link name="drone_arm_2">
     <inertial>
       <origin xyz="${arm_origin}" rpy="${zero_rpy}"/>
@@ -139,5 +139,5 @@
     </collision>
   </link>
-  <link name="copter_arm_3">
+  <link name="drone_arm_3">
     <inertial>
       <origin xyz="${arm_origin}" rpy="${zero_rpy}"/>
@@ -159,5 +159,5 @@
     </collision>
   </link>
-  <link name="copter_arm_4">
+  <link name="drone_arm_4">
     <inertial>
       <origin xyz="${arm_origin}" rpy="${zero_rpy}"/>
@@ -180,6 +180,6 @@
   </link>
   <!-- #endregion -->
-  <!-- #region Copter Props -->
-  <link name="copter_prop_1">
+  <!-- #region Drone Props -->
+  <link name="drone_prop_1">
     <inertial>
       <origin xyz="${prop_origin}" rpy="${zero_rpy}"/>
@@ -201,5 +201,5 @@
     </collision>
   </link>
-  <link name="copter_prop_2">
+  <link name="drone_prop_2">
     <inertial>
       <origin xyz="${prop_origin}" rpy="${zero_rpy}"/>
@@ -221,5 +221,5 @@
     </collision>
   </link>
-  <link name="copter_prop_3">
+  <link name="drone_prop_3">
     <inertial>
       <origin xyz="${prop_origin}" rpy="${zero_rpy}"/>
@@ -241,5 +241,5 @@
     </collision>
   </link>
-  <link name="copter_prop_4">
+  <link name="drone_prop_4">
     <inertial>
       <origin xyz="${prop_origin}" rpy="${zero_rpy}"/>
@@ -262,6 +262,6 @@
   </link>
   <!-- #endregion -->
-  <!-- #region Copter Camera -->
-   <link name="copter_camera">
+  <!-- #region Drone Camera -->
+   <link name="drone_camera">
     <inertial>
       <origin xyz="${camera_origin}" rpy="${zero_rpy}"/>
@@ -285,21 +285,21 @@
   <!-- #region Arm Joints -->
   <joint name="base_to_arm_1" type="fixed">
-    <parent link="copter_base"/>
-    <child link="copter_arm_1"/>
+    <parent link="drone_base"/>
+    <child link="drone_arm_1"/>
     <origin xyz="${base_radius*cos(pi/4)} ${base_radius*sin(pi/4)} ${arm_joint_zorigin}" rpy="${-pi/2} 0.0 ${-pi/4+0*pi/2}"/>
   </joint>
   <joint name="base_to_arm_2" type="fixed">
-    <parent link="copter_base"/>
-    <child link="copter_arm_2"/>
+    <parent link="drone_base"/>
+    <child link="drone_arm_2"/>
     <origin xyz="${base_radius*cos(3*pi/4)} ${base_radius*sin(3*pi/4)} ${arm_joint_zorigin}" rpy="${-pi/2} 0.0 ${-pi/4+pi/2}"/>
   </joint>
   <joint name="base_to_arm_3" type="fixed">
-    <parent link="copter_base"/>
-    <child link="copter_arm_3"/>
+    <parent link="drone_base"/>
+    <child link="drone_arm_3"/>
     <origin xyz="${base_radius*cos(5*pi/4)} ${base_radius*sin(5*pi/4)} ${arm_joint_zorigin}" rpy="${-pi/2} 0.0 ${-pi/4+2*pi/2}"/>
   </joint>
   <joint name="base_to_arm_4" type="fixed">
-    <parent link="copter_base"/>
-    <child link="copter_arm_4"/>
+    <parent link="drone_base"/>
+    <child link="drone_arm_4"/>
     <origin xyz="${base_radius*cos(7*pi/4)} ${base_radius*sin(7*pi/4)} ${arm_joint_zorigin}" rpy="${-pi/2} 0.0 ${-pi/4+3*pi/2}"/>
   </joint>
@@ -307,21 +307,21 @@
   <!-- #region Prop Joints -->
   <joint name="arm_1_to_prop_1" type="fixed">
-    <parent link="copter_arm_1"/>
-    <child link="copter_prop_1"/>
+    <parent link="drone_arm_1"/>
+    <child link="drone_prop_1"/>
     <origin xyz="${prop_joint_origin}" rpy="${prop_joint_rpy}"/>
   </joint>
   <joint name="arm_2_to_prop_2" type="fixed">
-    <parent link="copter_arm_2"/>
-    <child link="copter_prop_2"/>
+    <parent link="drone_arm_2"/>
+    <child link="drone_prop_2"/>
     <origin xyz="${prop_joint_origin}" rpy="${prop_joint_rpy}"/>
   </joint>
   <joint name="arm_3_to_prop_3" type="fixed">
-    <parent link="copter_arm_3"/>
-    <child link="copter_prop_3"/>
+    <parent link="drone_arm_3"/>
+    <child link="drone_prop_3"/>
     <origin xyz="${prop_joint_origin}" rpy="${prop_joint_rpy}"/>
   </joint>
   <joint name="arm_4_to_prop_4" type="fixed">
-    <parent link="copter_arm_4"/>
-    <child link="copter_prop_4"/>
+    <parent link="drone_arm_4"/>
+    <child link="drone_prop_4"/>
     <origin xyz="${prop_joint_origin}" rpy="${prop_joint_rpy}"/>
   </joint>
@@ -329,6 +329,6 @@
   <!-- #region Prop Joints -->
   <joint name="base_to_camera" type="fixed">
-    <parent link="copter_base"/>
-    <child link="copter_camera"/>
+    <parent link="drone_base"/>
+    <child link="drone_camera"/>
     <origin xyz="${camera_joint_origin}" rpy="${camera_joint_rpy}"/>
   </joint>
@@ -336,14 +336,14 @@
   <!-- #region Drake Commands -->
   <drake:collision_filter_group name="self_collision_ignore">
-    <drake:member link="copter_base"/>
-    <drake:member link="copter_arm_1"/>
-    <drake:member link="copter_arm_2"/>
-    <drake:member link="copter_arm_3"/>
-    <drake:member link="copter_arm_4"/>
-    <drake:member link="copter_prop_1"/>
-    <drake:member link="copter_prop_2"/>
-    <drake:member link="copter_prop_3"/>
-    <drake:member link="copter_prop_4"/>
-    <drake:member link="copter_camera"/>
+    <drake:member link="drone_base"/>
+    <drake:member link="drone_arm_1"/>
+    <drake:member link="drone_arm_2"/>
+    <drake:member link="drone_arm_3"/>
+    <drake:member link="drone_arm_4"/>
+    <drake:member link="drone_prop_1"/>
+    <drake:member link="drone_prop_2"/>
+    <drake:member link="drone_prop_3"/>
+    <drake:member link="drone_prop_4"/>
+    <drake:member link="drone_camera"/>
     <drake:ignored_collision_filter_group name="self_collision_ignore"/>
   </drake:collision_filter_group>
